Commit message: herp

File: notes/arm/arm.urdf (robot description, URDF)
Before this commit: robot tidybot arm, 6 links, 5 joints
Links:
- link base_link: geometry visual mesh filename=https://github.com/G9-Robotikk-2023-hvl/Tidybot/blob/main/n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

Commit message: derp

File: notes/arm/arm.urdf (robot description, URDF)
Before this commit: robot tidybot arm, 6 links, 5 joints
Links:
- added link link_end_point; visual cylinder length=0.1 radius=0.1
- link base_link: geometry visual box size=0.56 0.56 0.1
Joints:
- added joint joint_end: type fixed, parent link_end, child link_end_point, origin xyz=0 -0.28 0.5 rpy=0 0 0
- joint joint3: origin xyz=0 -5 0 rpy=0 1.5708 1.5708 -> xyz=0 -5 0 rpy=1.5708 0 0
